Commit message: new model

File: mp_500/mp_500.urdf (robot description, URDF)
Before this commit: robot mp_400, 4 links, 3 joints
Links:
- removed link back_wheel
- link base_link: geometry collision cylinder length=0.35 radius=0.3; visual cylinder length=0.29 radius=0.255
- link left_wheel: geometry collision cylinder length=0.03 radius=0.075; visual cylinder length=0.03 radius=0.075
Joints:
- removed joint base_to_back_wheel
