Commit message: mpo_500 robot model fixed

File: mpo_500/mpo_500.urdf (robot description, URDF)
Before this commit: robot mpo_500, 7 links, 6 joints
Links:
- removed link laserback_link
- removed link laserfront_link
Joints:
- removed joint laserback_joint
- removed joint laserfront_joint
- joint wheel_back_left_joint: type continuous -> fixed
- joint wheel_back_right_joint: type continuous -> fixed
- joint wheel_front_left_joint: type continuous -> fixed
- joint wheel_front_right_joint: type continuous -> fixed

Commit message: updated mpo_500 to have meshes + gazebo bindings * added sick laser gazebo plugin descriptions * reorganized xacro files * added testing directory * added meshes * added install locations * removed duplicate macros

File: mpo_500/mpo_500.urdf (robot description, URDF)
Before this commit: robot mpo_500, 5 links, 4 joints
Links:
- link base_link: geometry collision box size=0.769 0.51 0.307; visual mesh filename=package://neo_robot_descriptions/mpo_500/meshes/MPO-500-BOD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
- link wheel_back_left_link: geometry collision cylinder length=0.1 radius=0.12; visual mesh filename=package://neo_robot_descriptions/mpo_500/meshes/MPO-500-WHE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
- link wheel_back_right_link: geometry collision cylinder length=0.1 radius=0.12; visual mesh filename=package://neo_robot_descriptions/mpo_500/meshes/MPO-500-WHE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
- link wheel_front_left_link: geometry collision cylinder length=0.1 radius=0.12; visual mesh filename=package://neo_robot_descriptions/mpo_500/meshes/MPO-500-WHE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
- link wheel_front_right_link: geometry collision cylinder length=0.1 radius=0.12; visual mesh filename=package://neo_robot_descriptions/mpo_500/meshes/MPO-500-WHE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

File: mpo_500/xacro_macros/materials.urdf.xacro (robot description, xacro)
@@ -1,22 +1,27 @@
 <?xml version="1.0"?>
-    <material name="Black">
+<robot>
+    <material name="Neobotix/Black">
         <color rgba="0.0 0.0 0.0 1.0"/>
     </material>
-    <material name="Blue">
+    <material name="Neobotix/Blue">
         <color rgba="0.0 0.0 0.8 1.0"/>
     </material>
-    <material name="Green">
+    <material name="Neobotix/Green">
         <color rgba="0.0 0.8 0.0 1.0"/>
     </material>
-    <material name="Grey">
+    <material name="Neobotix/Grey">
         <color rgba="0.7 0.7 0.7 1.0"/>
     </material>
-    <material name="Grey2">
+    <material name="Neobotix/Grey2">
         <color rgba="0.9 0.9 0.9 1.0"/>
     </material>
-    <material name="Red">
+    <material name="Neobotix/Red">
         <color rgba="0.8 0.0 0.0 1.0"/>
     </material>
-    <material name="White">
+    <material name="Neobotix/White">
         <color rgba="1.0 1.0 1.0 1.0"/>
     </material>
+    <material name="Neobotix/Yellow">
+        <color rgba="1.0 1.0 0 10" />
+    </material>
+</robot>

File: mpo_500/xacro_macros/mpo_500_base.urdf.xacro (robot description, xacro)
@@ -1,124 +1,31 @@
 <?xml version="1.0"?>
 <robot xmlns:xacro="http://www.ros.org/wiki/xacro" name="mpo_500">
-<!-- Sensors -->
-<macro name="sick_s300_laser_v0" params="name parent *origin">
-    <joint name="${name}_joint" type="fixed">
-      <axis xyz="0 1 0" />
-      <insert_block name="origin" />
-      <parent link="${parent}"/>
-      <child link="${name}_link"/>
-    </joint>
-    <link name="${name}_link" type="laser">
-      <inertial>
-        <mass value="0.001" />
-        <origin xyz="0 0 0" rpy="0 0 0" />
-        <inertia ixx="0.0001" ixy="0" ixz="0" iyy="0.000001" iyz="0" izz="0.0001" />
-      </inertial>
-      <visual>
-        <origin xyz="0 0 0" rpy="0 0 0" />
-        <geometry>
-          <box size="0.001 0.001 0.001" />
-        </geometry>
-        <material name="Red" />
-      </visual>
-      <collision>
-        <origin xyz="0 0 0" rpy="0 0 0" />
-        <geometry>
-          <box size=".001 .001 .001" />
-        </geometry>
-      </collision>
-    </link>
-  </macro>
-<!-- Wheel Macro -->
-<xacro:macro name="omni_wheel_250" params="name parent *origin">
- <joint name="${name}_joint" type="continuous">
-  <insert_block name="origin" />
-  <axis xyz="0 1 0" />
-  <joint_properties damping="0.0" friction="0.0" />
-  <parent link="${parent}" />
-  <child link="${name}_link" />
- </joint>
- <link name="${name}_link" type="wheel">
-  <inertial>
-    <mass value="0.001" />
-    <origin xyz="0 0 0" rpy="0 0 0" />
-    <inertia ixx="0.0001" ixy="0" ixz="0" iyy="0.000001" iyz="0" izz="0.0001" />
-  </inertial>
-  <visual>
-   <origin xyz="0 0 0" rpy="1.59 0 0" />
-   <geometry>
-	<cylinder radius="0.12" length="0.1"/>
-   </geometry>
-   <material name="Black" />
-  </visual>
-  <collision>
-   <origin xyz="0 0 0" rpy="1.59 0 0" />
-   <geometry>
-	<cylinder radius="0.12" length="0.1"/>
-   </geometry>
-  </collision>
- </link>
-</xacro:macro>
-<!-- Materials -->
-<material name="Black">
-        <color rgba="0.0 0.0 0.0 1.0"/>
-    </material>
-    <material name="Blue">
-        <color rgba="0.0 0.0 0.8 1.0"/>
-    </material>
-    <material name="Green">
-        <color rgba="0.0 0.8 0.0 1.0"/>
-    </material>
-    <material name="Grey">
-        <color rgba="0.7 0.7 0.7 1.0"/>
-    </material>
-    <material name="Grey2">
-        <color rgba="0.9 0.9 0.9 1.0"/>
-    </material>
-    <material name="Red">
-        <color rgba="0.8 0.0 0.0 1.0"/>
-    </material>
-    <material name="White">
-        <color rgba="1.0 1.0 1.0 1.0"/>
-    </material>
-<!-- ROBOT -->
-<!-- BODY -->
-  <link name="base_link">
-    <inertial>
-      <mass value="20" />
-      <origin xyz="0 0 0" />
-      <inertia ixx="1.0" ixy="0.0" ixz="0.0"
-               iyy="1.0" iyz="0.0"
-               izz="1.0" />
-    </inertial>
-    <visual>
-       <origin xyz="0. 0. 0.2" rpy="0 0 0" />
-       <geometry><box size="0.68 0.41 0.25"/></geometry>
-       <material name="Grey" />
-    </visual>
-    <collision>
-       <origin xyz="0. 0. 0.2" rpy="0 0 0" />
-       <geometry><box size="0.68 0.41 0.25"/></geometry>
-    </collision>
-  </link>
-<!-- WHEELS -->
-  <omni_wheel_250 name="wheel_front_left" parent="base_link">
-     <origin xyz="0.25 0.28 0.13" rpy="0 0 0" />
-  </omni_wheel_250>
-  <omni_wheel_250 name="wheel_front_right" parent="base_link">
-     <origin xyz="0.25 -0.28 0.13" rpy="0 0 0" />
-  </omni_wheel_250>
-  <omni_wheel_250 name="wheel_back_left" parent="base_link">
-      <origin xyz="-0.25 0.28 0.13" rpy="0 0 0" />
-  </omni_wheel_250>
-  <omni_wheel_250 name="wheel_back_right" parent="base_link">
-      <origin xyz="-0.25 -0.28 0.13" rpy="0 0 0" />
-  </omni_wheel_250>
-<!-- Laser Scanner -->
-  <sick_s300_laser_v0 name="laserfront" parent="base_link">
-    <origin xyz="0.39 0 0" rpy="0 0 0" />
-  </sick_s300_laser_v0>
-  <sick_s300_laser_v0 name="laserback" parent="base_link">
-    <origin xyz="-0.39 0 0" rpy="0 0 3.14" />
-  </sick_s300_laser_v0>
+    <xacro:include filename="$(find neo_robot_descriptions)/mpo_500/xacro_macros/sick_s300_laser.urdf.xacro" />
+    <xacro:include filename="$(find neo_robot_descriptions)/mpo_500/xacro_macros/omni_wheel.urdf.xacro" />
+    <xacro:include filename="$(find neo_robot_descriptions)/mpo_500/xacro_macros/materials.urdf.xacro"/>
+    <xacro:include filename="$(find neo_robot_descriptions)/mpo_500/xacro_macros/mpo_500_body.urdf.xacro"/>
+    <xacro:macro name="mpo_500" params="name">
+        <!-- BASE -->
+        <xacro:mpo_500_base name="${name}_base_link" />
+        <!-- WHEELS -->
+        <xacro:omni_wheel_250 name="${name}_wheel_front_left" parent="${name}_base_link">
+            <origin xyz="0.25 0.28 0.13" rpy="0 0 0" />
+        </xacro:omni_wheel_250>
+        <xacro:omni_wheel_250 name="${name}_wheel_front_right" parent="${name}_base_link">
+            <origin xyz="0.25 -0.28 0.13" rpy="0 0 0" />
+        </xacro:omni_wheel_250>
+        <xacro:omni_wheel_250 name="${name}_wheel_back_left" parent="${name}_base_link">
+            <origin xyz="-0.25 0.28 0.13" rpy="0 0 0" />
+        </xacro:omni_wheel_250>
+        <xacro:omni_wheel_250 name="${name}_wheel_back_right" parent="${name}_base_link">
+            <origin xyz="-0.25 -0.28 0.13" rpy="0 0 0" />
+        </xacro:omni_wheel_250>
+        <!-- LASER SCANNER -->
+        <xacro:sick_s300_laser_v0 name="${name}_laserfront" parent="${name}_base_link" ros_topic="${name}/laserfront/scan">
+            <origin xyz="0.442 0 0.333" rpy="0 0 0" />
+        </xacro:sick_s300_laser_v0>
+        <xacro:sick_s300_laser_v0 name="${name}_laserback" parent="${name}_base_link" ros_topic="${name}/laserback/scan">
+            <origin xyz="-0.442 0 0.333" rpy="0 0 3.14" />
+        </xacro:sick_s300_laser_v0>
+    </xacro:macro>
 </robot>

File: mpo_500/xacro_macros/omni_wheel.urdf.xacro (robot description, xacro)
@@ -1,30 +1,37 @@
 <?xml version="1.0"?>
-<xacro:macro name="omni_wheel_250" params="suffix parent *origin">
- <joint name="${suffix}_joint" type="continuous">
-  <insert_block name="origin" />
-  <axis xyz="0 1 0" />
-  <joint_properties damping="0.0" friction="0.0" />
-  <parent link="${parent}_link" />
-  <child link="${suffix}_link" />
- </joint>
- <link name="${suffix}_link" type="wheel">
-  <inertial>
-    <mass value="0.001" />
-    <origin xyz="0 0 0" rpy="0 0 0" />
-    <inertia ixx="0.0001" ixy="0" ixz="0" iyy="0.000001" iyz="0" izz="0.0001" />
-  </inertial>
-  <visual>
-   <origin xyz="0 0 0" rpy="1.59 0 0" />
-   <geometry>
-	<cylinder radius="0.12" length="0.1"/>
-   </geometry>
-   <material name="Black" />
-  </visual>
-  <collision>
-   <origin xyz="0 0 0" rpy="1.59 0 0" />
-   <geometry>
-	<cylinder radius="0.12" length="0.1"/>
-   </geometry>
-  </collision>
- </link>
-</xacro:macro>
+<robot xmlns:xacro="http://www.ros.org/wiki/xacro" name="mpo_500">
+  <xacro:macro name="omni_wheel_250" params="name parent *origin">
+   <joint name="${name}_joint" type="fixed">
+    <insert_block name="origin" />
+    <axis xyz="0 1 0" />
+    <joint_properties damping="0.0" friction="0.0" />
+    <parent link="${parent}" />
+    <child link="${name}_link" />
+   </joint>
+   <link name="${name}_link" type="wheel">
+    <inertial>
+      <mass value="0.001" />
+      <origin xyz="0 0 0" rpy="0 0 0" />
+      <inertia ixx="0.0001" ixy="0" ixz="0" iyy="0.000001" iyz="0" izz="0.0001" />
+    </inertial>
+    <visual>
+     <origin xyz="0 0 0" rpy="0 0 1.571" />
+     <geometry>
+        <mesh filename="package://neo_robot_descriptions/mpo_500/meshes/MPO-500-WHEEL.STL"/>
+     </geometry>
+     <material name="Neobotix/Black" />
+    </visual>
+    <collision>
+     <origin xyz="0 0 0" rpy="1.59 0 0" />
+     <geometry>
+        <cylinder radius="0.12" length="0.1"/>
+     </geometry>
+    </collision>
+   </link>
+    <gazebo reference="${name}_link">
+        <gravity>true</gravity>
+        <self_collide>false</self_collide>
+        <material value="Gazebo/Black"/>
+    </gazebo>
+  </xacro:macro>
+</robot>

File: mpo_500/xacro_macros/sick_s300_laser.urdf.xacro (robot description, xacro)
@@ -1,9 +1,9 @@
 <?xml version="1.0"?>
-<robot>
-  <macro name="sick_s300_laser_v0" params="name parent *origin ros_topic update_rate min_angle max_angle">
+<robot xmlns:xacro="http://www.ros.org/wiki/xacro" name="mpo_500">
+  <xacro:macro name="sick_s300_laser_v0" params="name parent *origin ros_topic">
     <joint name="${name}_joint" type="fixed">
       <axis xyz="0 1 0" />
       <insert_block name="origin" />
-      <parent link="${parent}_link"/>
+      <parent link="${parent}"/>
       <child link="${name}_link"/>
     </joint>
@@ -15,17 +15,55 @@
       </inertial>
       <visual>
-        <origin xyz="0 0 0" rpy="0 0 0" />
+        <origin xyz="0 0 0" rpy="0 0 -1.57" />
         <geometry>
-          <box size="0.001 0.001 0.001" />
+          <mesh filename="package://neo_robot_descriptions/mpo_500/meshes/MPO-500-SICK.STL" />
         </geometry>
-        <material name="Red" />
+        <material name="Neobotix/Yellow" />
       </visual>
       <collision>
         <origin xyz="0 0 0" rpy="0 0 0" />
         <geometry>
-          <box size=".001 .001 .001" />
+          <cylinder length="0.154" radius="0.053" />
         </geometry>
       </collision>
     </link>
-  </macro>
+    <gazebo reference="${name}_link">
+      <gravity>true</gravity>
+      <self_collide>false</self_collide>
+      <material value="Gazebo/Yellow"/>
+      <sensor type="ray" name="${name}_sensor">
+          <pose>0 0 0 0 0 0</pose>
+          <visualize>false</visualize>
+          <update_rate>40</update_rate>
+          <ray>
+            <scan>
+              <horizontal>
+                <samples>720</samples>
+                <resolution>1</resolution>
+                <min_angle>-1.570796</min_angle>
+                <max_angle>1.570796</max_angle>
+              </horizontal>
+            </scan>
+            <range>
+              <min>0.10</min>
+              <max>30.0</max>
+              <resolution>0.01</resolution>
+            </range>
+            <noise>
+              <type>gaussian</type>
+              <!-- Noise parameters based on published spec for Hokuyo laser
+                   achieving "+-30mm" accuracy at range < 10m.  A mean of 0.0m and
+                   stddev of 0.01m will put 99.7% of samples within 0.03m of the true
+                   reading. -->
+              <mean>0.0</mean>
+              <stddev>0.01</stddev>
+            </noise>
+          </ray>
+          <plugin name="${name}_controller" filename="libgazebo_ros_laser.so">
+            <topicName>${ros_topic}</topicName>
+            <frameName>${name}_link</frameName>
+          </plugin>
+        </sensor>
+    </gazebo>
+  </xacro:macro>
 </robot>
